Commit message: fixes for sim env

File: src/pybullet_robot/robots/bullet_panda/models/panda_arm_with_block.urdf (robot description, URDF)
Before this commit: robot panda, 9 links, 8 joints
Links:
- link ee_block: mass 1.0 -> 0.5; geometry collision box size=0.2 0.1 0.07; visual box size=0.2 0.1 0.07
